File: kicad/enclosure_sys/enclosure_sys.kicad_sch (KiCad schematic)
At the start: 0 parts

Commit message: fix fans
Parts:
- added A1: RaspberryPi_Pico_W, Module:RaspberryPi_Pico_W_SMD_HandSolder, symbol MCU_Module:RaspberryPi_Pico_W
- added D1: LIGHT, symbol Device:LED
- added J1: pmod oled, symbol Connector_Generic:Conn_02x06_Odd_Even
- added M1, M2: Fan, symbol Motor:Fan
- added Q1, Q2: NPN, symbol Simulation_SPICE:NPN
- added R1, R2: 10 Ohm, symbol Device:R
- added R3: 5kOhm, symbol Device:R
- added SW1: SW_SPST, symbol Switch:SW_SPST
- added U1: DS18B20, Package_TO_SOT_THT:TO-92_Inline, symbol Sensor_Temperature:DS18B20
Connections:
- new net: M1.2 (-), Q2.3 (E)
- new net: D1.2 (A), SW1.2 (B)
- new net: Q1.2 (B), R1.1
- new net: A1.20 (GPIO15), R1.2
- new net: A1.19 (GPIO14), R2.2
- new net: M2.2 (-), Q1.3 (E)
- new net: Q2.2 (B), R2.1
- new net 3V3: A1.36 (3V3), R3.2, U1.3 (V_{DD})
- new net CS: A1.22 (GPIO17), J1.1 (Pin_1)
- new net DATA_TEMP: A1.34 (GPIO28_ADC2), R3.1, U1.2 (DQ)
- new net D/C: A1.21 (GPIO16), J1.7 (Pin_7)
- new net GND: A1.13 (GND), A1.18 (GND), A1.23 (GND), A1.28 (GND), A1.3 (GND), A1.38 (GND), A1.8 (GND), D1.1 (K), J1.5 (Pin_5), Q1.1 (C), Q2.1 (C), U1.1 (GND)
- new net MOSI: A1.25 (GPIO19), J1.2 (Pin_2)
- new net RESET: A1.29 (GPIO22), J1.8 (Pin_8)
- new net SCLK: A1.24 (GPIO18), J1.4 (Pin_4)
- new net VSYS: A1.39 (VSYS), J1.6 (Pin_6), M1.1 (+), M2.1 (+), SW1.1 (A)
Other:
- note added: "fans"
